Commit message: change modele

File: urdf/aiibot.urdf (robot description, URDF)
Before this commit: robot aiibot, 12 links, 11 joints
Joints:
- joint base_liser_joint: origin xyz=-0.100 0 0.2 -> xyz=-0.250 0 0.2 rpy=0 0 3.1415927

Commit message: change model

File: urdf/aiibot.urdf (robot description, URDF)
Before this commit: robot aiibot, 12 links, 11 joints
Links:
- link base_link: geometry visual box size=0.51 0.426 .003
- link laser: geometry visual cylinder length=0.025 radius=0.035
- link lidar_up: geometry visual cylinder length=0.035 radius=0.01
- link right_front_wheel: geometry visual cylinder length=0.015 radius=0.048
- link shelf_left: geometry visual box size=0.25 0.001 .09
- link shelf_lidar_front: geometry visual box size=0.001 0.10 .07
- link shelf_lidar_top: geometry visual box size=0.1 0.1 .001
- link shelf_right: geometry visual box size=0.25 0.001 .09
- link shelf_top: geometry visual box size=0.25 0.30 .001
Joints:
- joint base_liser_joint: origin xyz=-0.250 0 0.2 rpy=0 0 3.1415927 -> xyz=0 0 0.03 rpy=0 0 3.1415927; parent base_link -> lidar_up
- joint left_front_wheel_joint: origin xyz=0 0.24 -0.025 rpy=0 1.57075 1.57075 -> xyz=0 0.2255 -0.0255 rpy=0 1.57075 1.57075
- joint lidar_up_joint: origin xyz=-0.100 0 0.172 -> xyz=0 0 0.018; parent base_link -> shelf_lidar_top
- joint right_front_wheel_joint: origin xyz=0 -0.24 -0.025 rpy=0 1.57075 1.57075 -> xyz=0 -0.2255 -0.0255 rpy=0 1.57075 1.57075
- joint shelf_left_joint: origin xyz=-0.13 -0.149 0.04 rpy=0 0 0 -> xyz=-0.17 -0.1495 0.0465 rpy=0 0 0
- joint shelf_lidar_front_joint: origin xyz=-0.041 0 0.12 rpy=0 0 0 -> xyz=-0.0845 0 0.0355 rpy=0 0 0; parent base_link -> shelf_top
- joint shelf_lidar_top_joint: origin xyz=-0.09 0 0.16 rpy=0 0 0 -> xyz=0.0495 0 0.0345 rpy=0 0 0; parent base_link -> shelf_lidar_front
- joint shelf_right_joint: origin xyz=-0.13 0.149 0.04 rpy=0 0 0 -> xyz=-0.17 0.1495 0.0465 rpy=0 0 0
- joint shelf_top_joint: origin xyz=-0.13 0 0.08 rpy=0 0 0 -> xyz=-0.17 0 0.091 rpy=0 0 0

Commit message: modify urdf

File: urdf/aiibot.urdf (robot description, URDF)
Before this commit: robot aiibot, 12 links, 11 joints
Links:
- added link kinect; visual box size=0.035 0.18 .02
- added link kinect_shelf; visual box size=0.04 0.1 .18
- added link kinect_up; visual cylinder length=0.02 radius=0.005
Joints:
- added joint kinect_joint: type continuous, parent kinect_up, child kinect, origin xyz=0 0 0.02 rpy=0 0 0, axis 0 0 1, limit effort=100 velocity=100
- added joint kinect_shelf_joint: type continuous, parent shelf_lidar_front, child kinect_shelf, origin xyz=-0.0205 0 0.055 rpy=0 0 0, axis 0 0 1, limit effort=100 velocity=100
- added joint kinect_up_joint: type fixed, parent kinect_shelf, child kinect_up, origin xyz=0 0 0.10
